Commit message: - left / right finger tip state

File: assets/urdf/ur_description/urdf/ur3e_robotiq_2f_85.urdf (robot description, URDF)
Before this commit: robot ur3e_robotiq, 22 links, 21 joints
Links:
- added link ur3e_grip_site
Joints:
- added joint ur3e_grip_tool0: type fixed, parent ur3e_tool0, child ur3e_grip_site, origin xyz=0 0 0.127 rpy=0 0 0
