Commit message: - define allegro hand grip site

File: assets/urdf/ur_with_allegro_hand_description/urdf/ur3_allegro_right_hand.urdf (robot description, URDF)
Before this commit: robot ur_robot, 35 links, 34 joints
Links:
- added link allegro_grip_site
Joints:
- added joint allegro_grip_tool0: type fixed, parent tool0, child allegro_grip_site, origin xyz=0 0 0.0625 rpy=0 0 0
