Commit message: - model path including year-month - bimanual hands' palm index offset - minor updates...

File: assets/urdf/ur_with_allegro_hand_description/urdf/ur3_allegro_left_hand.urdf (robot description, URDF)
Before this commit: robot ur_robot, 36 links, 35 joints
Joints:
- joint allegro_grip_tool0: origin xyz=0 0 0.0625 rpy=0 0 0 -> xyz=0 0.02 0.0625 rpy=0 0 0

File: assets/urdf/ur_with_allegro_hand_description/urdf/ur3_allegro_right_hand.urdf (robot description, URDF)
Before this commit: robot ur_robot, 36 links, 35 joints
Joints:
- joint allegro_grip_tool0: origin xyz=0 0 0.0625 rpy=0 0 0 -> xyz=0 0.02 0.0625 rpy=0 0 0
