Commit message: Got environment setup

File: assets/urdf/ycb/011_banana/011_banana.urdf (robot description, URDF)
Before this commit: robot banana, 1 links, 0 joints
Links:
- link banana: geometry collision mesh filename=/home/sankalp/ws_spot_catching/src/BimanualDexCatch/assets/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 scale=0.01 0.01 0.01; visual mesh filename=/home/sankalp/ws_spot_catching/src/BimanualDexCatch/assets/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 scale=0.01 0.01 0.01
