Commit message: Trying to addpybullet for contacts

File: assets/urdf/football.urdf (robot description, URDF)
Before this commit: robot football, 1 links, 0 joints
Links:
- link football: geometry collision mesh filename=/home/sankalp/ws_spot_catching/src/BimanualDexCatch/assets/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 scale=0.8 0.8 0.8; visual mesh filename=/home/sankalp/ws_spot_catching/src/BimanualDexCatch/assets/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 scale=0.8 0.8 0.8

Commit message: Run on lambda while editing rewards

File: assets/urdf/football.urdf (robot description, URDF)
Before this commit: robot football, 1 links, 0 joints
Links:
- link football: geometry collision mesh filename=/home/sankalp/ws_spot_catching/src/BimanualDexCatch/assets/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 scale=0.55 0.55 0.55; visual mesh filename=/home/sankalp/ws_spot_catching/src/BimanualDexCatch/assets/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 scale=0.55 0.55 0.55
